File: Nixie Wrist Clock V1.sch (EAGLE design)
At the start: 39 parts, among them Q1 310mA/60V/1.6Ω, Q2 310mA/60V/1.6Ω, Q3 310mA/60V/1.6Ω, Q4 310mA/60V/1.6Ω, Q5 310mA/60V/1.6Ω, U2 NRF52832, X3 32MHz, X4 32.768kHz

Commit message: Update#7
5V Boost Regulator Added
Parts:
- added C10: 10uF, rcl:CPOL-EUSMCA
- added C11: 22uF, rcl:CPOL-EUSMCB
- added C5, C6, C7: 100nF, Nordic_nRF:CAPACITOR_0603_N
- added C9: 100pF, Nordic_nRF:CAPACITOR_0603_N
- added R12: 6.65K, rcl:R-EU_R0603
- added R13: 768K, rcl:R-EU_R0603
- added R14: 243K, rcl:R-EU_R0603
- added R15: 868K, rcl:R-EU_R0603
- added U$4: TPS61252DSGR, Alp-Special:TPS61252DSGR
- added U$5: FPI-SERIES-INDUCTOR0302, Alp-Special:FPI-SERIES-INDUCTOR0302
Connections:
- new net 5V-ENA: U$4.EN
- new net N$10: R15.2, U$4.PG
- new net N$14: C9.2, R13.2, R14.1, U$4.FB
- new net N$6: U$4.SW, U$5.2
- new net N$8: R12.1, U$4.ILIM
- net +5V: now also C11.+, C9.1, R13.1, R15.1, U$4.VOUT
- net GND: now also C10.-, C11.-, R12.2, R14.2, U$4.GND
- net VCC: now also C10.+, U$4.VIN, U$5.1
Other:
- note added: "C10"
- note added: "C11"
- note added: "Inductor"
- note added: "https://www.ozdisan.com/pasif-komponentler/induktorler/sabit-induktor/FPI0302-2R2M"
- note added: "https://www.ozdisan.com/pasif-komponentler/kondansatorler/tantal-kondansatorler/T491A106K010AT"
- note added: "https://www.ozdisan.com/pasif-komponentler/kondansatorler/tantal-kondansatorler/TAJB226K016RNJ"

Commit message: Update#7
Parts:
- removed C5, C6, C7: 100nF, Nordic_nRF:CAPACITOR_0603_N
- removed R11: 10K, rcl:R-EU_R0603
Changed lines of the file:
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@@
 <part name="U$3" library="Alp-Special" deviceset="TLV70233" device="SOT23-5"/>
 <part name="C3" library="Nordic_nRF" deviceset="CAPACITOR" device="_0603_N" value="100nF"/>
-<part name="R11" library="rcl" library_urn="urn:adsk.eagle:library:334" deviceset="R-EU_" device="R0603" package3d_urn="urn:adsk.eagle:package:23555/3" value="10K"/>
 <part name="+3V11" library="supply1" library_urn="urn:adsk.eagle:library:371" deviceset="+3V3" device=""/>
 <part name="P+7" library="supply1" library_urn="urn:adsk.eagle:library:371" deviceset="VCC" device=""/>
@@
 <part name="FRAME5" library="frames" library_urn="urn:adsk.eagle:library:229" deviceset="DINA4_L" device=""/>
 <part name="U$4" library="Alp-Special" deviceset="TPS61252DSGR" device=""/>
-<part name="C5" library="Nordic_nRF" deviceset="CAPACITOR" device="_0603_N" value="100nF"/>
-<part name="C6" library="Nordic_nRF" deviceset="CAPACITOR" device="_0603_N" value="100nF"/>
 <part name="U$5" library="Alp-Special" deviceset="FPI-SERIES-INDUCTOR" device="0302"/>
-<part name="C7" library="Nordic_nRF" deviceset="CAPACITOR" device="_0603_N" value="100nF"/>
 <part name="C9" library="Nordic_nRF" deviceset="CAPACITOR" device="_0603_N" value="100pF"/>
 <part name="R12" library="rcl" library_urn="urn:adsk.eagle:library:334" deviceset="R-EU_" device="R0603" package3d_urn="urn:adsk.eagle:package:23555/3" value="6.65K"/>
@@
 <attribute name="VALUE" x="75.184" y="107.061" size="1.778" layer="96"/>
 </instance>
-<instance part="R11" gate="G$1" x="124.46" y="132.08" smashed="yes" rot="R180">
-<attribute name="NAME" x="128.27" y="130.5814" size="1.778" layer="95" rot="R180"/>
-<attribute name="VALUE" x="128.27" y="135.382" size="1.778" layer="96" rot="R180"/>
-</instance>
 <instance part="+3V11" gate="G$1" x="86.36" y="116.84" smashed="yes" rot="R270">
 <attribute name="VALUE" x="81.28" y="119.38" size="1.778" layer="96"/>
@@
 <attribute name="VALUE" x="20.32" y="99.06" size="1.778" layer="96"/>
 </instance>
-<instance part="C5" gate="C$1" x="99.06" y="101.6" smashed="yes">
-<attribute name="NAME" x="100.584" y="101.981" size="1.778" layer="95"/>
-<attribute name="VALUE" x="100.584" y="96.901" size="1.778" layer="96"/>
-</instance>
-<instance part="C6" gate="C$1" x="96.52" y="111.76" smashed="yes">
-<attribute name="NAME" x="98.044" y="112.141" size="1.778" layer="95"/>
-<attribute name="VALUE" x="98.044" y="107.061" size="1.778" layer="96"/>
-</instance>
-<instance part="C7" gate="C$1" x="162.56" y="101.6" smashed="yes">
-<attribute name="NAME" x="164.084" y="101.981" size="1.778" layer="95"/>
-<attribute name="VALUE" x="164.084" y="96.901" size="1.778" layer="96"/>
-</instance>
 </instances>

Commit message: Update#7
Parts:
- added C5: 1pF, Nordic_nRF:CAPACITOR_0402_N
- C15: value 0.8pF -> 1pF
Connections:
- net GND: now also C5.2
- net RF: now also C5.1
Changed lines of the file:
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@@
 <part name="C13" library="Nordic_nRF" deviceset="CAPACITOR" device="_0603_N" value="12pF"/>
 <part name="C14" library="Nordic_nRF" deviceset="CAPACITOR" device="_0603_N" value="12pF"/>
-<part name="C15" library="Nordic_nRF" deviceset="CAPACITOR" device="_0402_N" value="0.8pF"/>
+<part name="C15" library="Nordic_nRF" deviceset="CAPACITOR" device="_0402_N" value="1pF"/>
 <part name="C16" library="Nordic_nRF" deviceset="CAPACITOR" device="_0603_N" value="100nF"/>
 <part name="C17" library="Nordic_nRF" deviceset="CAPACITOR" device="_0603_N" value="100nF"/>
@@
 <part name="P+10" library="supply1" library_urn="urn:adsk.eagle:library:371" deviceset="+5V" device=""/>
 <part name="P+11" library="supply1" library_urn="urn:adsk.eagle:library:371" deviceset="VCC" device=""/>
+<part name="C5" library="Nordic_nRF" deviceset="CAPACITOR" device="_0402_N" value="1pF"/>
+<part name="GND22" library="supply1" library_urn="urn:adsk.eagle:library:371" deviceset="GND" device=""/>
 </parts>
 <sheets>
@@
 <wire x1="43.18" y1="12.7" x2="43.18" y2="0" width="0.1524" layer="94"/>
 <text x="167.64" y="27.94" size="2.54" layer="94">MicroControler</text>
-<text x="185.42" y="78.74" size="1.778" layer="98">Anthenna Match 403 kılıfta</text>
+<text x="203.2" y="68.58" size="1.778" layer="98">Anthenna Match 403 kılıfta</text>
 <wire x1="10.16" y1="124.46" x2="10.16" y2="83.82" width="0.1524" layer="98"/>
 <wire x1="10.16" y1="83.82" x2="48.26" y2="83.82" width="0.1524" layer="98"/>
@@
 <attribute name="VALUE" x="134.62" y="137.16" size="1.778" layer="96" rot="R90"/>
 </instance>
+<instance part="C5" gate="C$1" x="195.58" y="81.28" smashed="yes">
+<attribute name="NAME" x="197.104" y="81.661" size="1.778" layer="95"/>
+<attribute name="VALUE" x="197.104" y="76.581" size="1.778" layer="96"/>
+</instance>
+<instance part="GND22" gate="1" x="195.58" y="71.12" smashed="yes" rot="MR0">
+<attribute name="VALUE" x="198.12" y="68.58" size="1.778" layer="96" rot="MR0"/>
+</instance>
 </instances>
 <busses>
@@
 <pinref part="C24" gate="C$1" pin="1"/>
 </segment>
+<segment>
+<pinref part="C5" gate="C$1" pin="2"/>
+<wire x1="195.58" y1="76.2" x2="195.58" y2="73.66" width="0.1524" layer="91"/>
+<pinref part="GND22" gate="1" pin="GND"/>
+</segment>
 </net>
 <net name="DEC1" class="0">
@@
 <segment>
 <pinref part="L2" gate="L$1" pin="2"/>
-<wire x1="193.04" y1="86.36" x2="205.74" y2="86.36" width="0.1524" layer="91"/>
+<wire x1="193.04" y1="86.36" x2="195.58" y2="86.36" width="0.1524" layer="91"/>
 <label x="198.12" y="86.36" size="1.778" layer="95"/>
-</segment>
-</net>
+<pinref part="C5" gate="C$1" pin="1"/>
+<wire x1="195.58" y1="86.36" x2="205.74" y2="86.36" width="0.1524" layer="91"/>
+<wire x1="195.58" y1="83.82" x2="195.58" y2="86.36" width="0.1524" layer="91"/>
+<junction x="195.58" y="86.36"/>
+</segment>
+</net>

Commit message: Update #8
Other:
- note added: "UPDATE #8"
Changed lines of the file:
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@@
 <?xml version="1.0" encoding="utf-8"?>
 <!DOCTYPE eagle SYSTEM "eagle.dtd">
-<eagle version="9.5.0">
+<eagle version="9.5.1">
 <drawing>
 <settings>
@@
 <wire x1="20.32" y1="12.7" x2="43.18" y2="12.7" width="0.1524" layer="94"/>
 <text x="2.54" y="10.16" size="1.778" layer="94">In Progress</text>
+<text x="20.32" y="165.1" size="6.4516" layer="91">UPDATE #8</text>
 </plain>
 <instances>

Commit message: Revert "Update #8"
This reverts commit 503de56c1cec5e58df481c359deaf8b3a9d703f1.
Other:
- note removed: "UPDATE #8"
Changed lines of the file:
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@@
 <?xml version="1.0" encoding="utf-8"?>
 <!DOCTYPE eagle SYSTEM "eagle.dtd">
-<eagle version="9.5.1">
+<eagle version="9.5.0">
 <drawing>
 <settings>
@@
 <wire x1="20.32" y1="12.7" x2="43.18" y2="12.7" width="0.1524" layer="94"/>
 <text x="2.54" y="10.16" size="1.778" layer="94">In Progress</text>
-<text x="20.32" y="165.1" size="6.4516" layer="91">UPDATE #8</text>
 </plain>
 <instances>
